File: Motion_Controller.sch (KiCad schematic (older format))
At the start: 0 parts

Commit message: continued work on the main processor
Parts:
- added B0_1/B0_0: HN1x3(B0_1:Open;B0_0:Close), symbol Connector_Generic:Conn_01x03
- added B1_1/B1_0: HN1x3(B1_1:Open;B1_0:Close), symbol Connector_Generic:Conn_01x03
- added C1, C15: 2.2uF/6.3V/10%/X5R/0603, symbol Device:C_Small
- added C10, C11, C12, C13, C14, C7, C8, C9, C?: 100nF/6.3V/20%/X5R/0603, symbol Device:C_Small
- added C16, C17, C2, C3, C4, C5, C6: 10uF/6.3V/20%/X5R/0603, symbol Device:C_Small
- added C19, C20: 27pF/50V/5%/CDG/0603, symbol Device:C_Small
- added C23, C?: 4.7pF/50V/0.1pF/C0G/0603, symbol Device:C_Small
- added C?: 100nF/650V/20%/Y5V/0603, symbol Device:C_Small
- added D?: BAT54C, Package_TO_SOT_SMD:SOT-23, symbol Diode:BAT54C
- added J?: 3V_BAT, symbol Connector:Conn_01x02_Male
- added JP?: AREF_EN, symbol Jumper:SolderJumper_2_Bridged
- added L?: INDUCTOR, symbol pspice:INDUCTOR
- added Q1: 12Mhz/30ppm/20pf, symbol Device:Crystal_Small
- added Q2: 32768Hz/6pF, symbol Device:Crystal_GND2_Small
- added R1: 0R, symbol Device:R_Small
- added R10, R7: NA, symbol Device:R_Small
- added R3, R5: 4.7k/5%/0603, symbol Device:R_Small
- added R4: 22R/5%/0603, symbol Device:R_Small
- added R6: 10k/5%/0603, symbol Device:R_Small
- added R8: 1.1k/1%/0603, symbol Device:R_Small
- added R9: 150R/5%/0603, symbol Device:R_Small
- added R?: R_Small, symbol Device:R_Small
- added SW?: RESET, symbol Switch:SW_Push
- added U?: STM32F407ZET6, lib_fp:LQFP-144_20x20mm_P0.5mm, symbol Motion_Controller:STM32F407ZET6
- added U?: LM810, Package_TO_SOT_SMD:SOT-23, symbol Power_Supervisor:LM810
Connections:
- new net: C15.1, U?.106 (VCAP_2)
- new net: C4.2, R1.2, R?.1, U?.143 (VDD_3)
- new net: C19.2, Q1.1, R7.1, U?.23 (PH0/OSC_IN)
- new net: R7.2, R9.1, U?.24 (PH1/OSC_OUT)
- new net: C?.2, R4.2, U?.32 (VREF+)
- new net: C1.1, U?.71 (VCAP_1)
- new net: C?.1, Q2.3, R10.2, U?.8 (PC14/OSC32_IN)
- new net: C23.1, Q2.1, R10.1, U?.9 (PC15/OSC32_OUT)
- new net: D?.1, J?.1 (Pin_1)
- new net: B0_1/B0_0.2 (Pin_2), R5.1
- new net: C?.2, R6.2, R8.1, SW?.1, U?.2 (RESET)
- new net: C20.2, Q1.2, R9.2
- new net: B1_1/B1_0.2 (Pin_2), R3.2
- new net +5V: B0_1/B0_0.1 (Pin_1), B1_1/B1_0.1 (Pin_1), C10.2, C11.2, C12.2, C13.2, C14.2, C16.1, C17.1, C2.2, C3.2, C5.2, C6.2, C7.2, C8.2, C9.2, C?.1, D?.2, L?.1, R1.1, R6.1, U?.108 (VDD_2), U?.121 (VDD_10), U?.131 (VDD_11), U?.144 (VDD_SA), U?.17 (VDD_5), U?.3 (VCC), U?.30 (VDD_12), U?.31 (VSSA), U?.39 (VDD_4), U?.52 (VDD_6), U?.62 (VDD_7), U?.72 (VDD_1), U?.84 (VDD_8), U?.95 (VDD_9)
- new net 3.3V_A: C16.2, C17.2, JP?.1 (A), L?.2, U?.33 (VDDA)
- new net AREF: JP?.2 (B), R4.1
- new net BOOT0: R5.2, U?.138 (BOOT0/VPP)
- new net GNDD: B0_1/B0_0.3 (Pin_3), B1_1/B1_0.3 (Pin_3), C1.2, C10.1, C11.1, C12.1, C13.1, C14.1, C15.2, C19.1, C2.1, C20.1, C23.2, C3.1, C4.1, C5.1, C6.1, C7.1, C8.1, C9.1, C?.1, C?.2, Q2.2, R?.2, SW?.2, U?.1 (GND), U?.107 (VSS_2), U?.120 (VSS_10), U?.130 (VSS_11), U?.16 (VSS_5), U?.38 (VSS_4), U?.51 (VSS_6), U?.61 (VSS_7), U?.83 (VSS_8), U?.94 (VSS_9)
- new net LED: U?.7 (PC13/RTC_AF1)
- new net PA0-WKUP: U?.34 (PA0/WKUP/USART2_CTS/USART4_TX/ETH_MII_CRS/TIM2_CH1_ETR/TIM5_CH1/TIM8_ETR/ADC123_CH0)
- new net PA1-D8-ETH_RMII_REF_CLK: U?.35 (PA1/USART2_RTS/USART4_RX/ETH_RMII_REF_CLK/ETH_MII_RX_CLK/TIM5_CH2/TIM2_CH2/ADC123_IN1)
- new net PA10-OTG1_FS_ID: U?.102 (PA10/USART1_RX/TIM1_CH3/OTG_FS_ID/DCMI_D1)
- new net PA11-OTG_FS_DM: U?.103 (PA11/USART1_CTS/CAN1_RX/TIM1_CH4/OTG_FS_DM)
- new net PA12-OTG_FS_DP: U?.104 (PA12/USART1_RTS/CAN1_TX/TIM1_ETR/OTG_FS_DP)
- new net PA13-TMS: U?.105 (PA13/JTMS-SWDIO)
- new net PA14-TCK: U?.109 (PA14/JTCK-SWCLK)
- new net PA15-TDI: U?.110 (PA15/JTDI/SPI3_NSS/I2S3_WS/TIM2_CH1_ETR/SPI1_NSS)
- new net PA2-ETH_RMII_MDIO: U?.36 (PA2/USART2_TX/TIM5_CH3/TIM9_CH1/TIM2_CH3/ETH_MDIO/ADC123_IN2)
- new net PA3-ETH_RMII_MDINT: U?.37 (PA3/USART2_RX/TIM5_CH4/TIM9_CH2/TIM2_CH4/OTG_HS_ULPI_D0/ETH_MII_COL/ADC123_IN3)
- new net PA4-D10-SPI1_NSS: U?.40 (PA4/SPI1_NSS/SPI3_NSS/USART2_CK/DCMI_HSYNC/OTG_HS_SOF/I2S3_WS/ADC12_IN4/DAC1_OUT)
- new net PA5-D13-SPI1_SCK: U?.41 (PA5/SPI1_SCK/OTG_HS_ULPI_CK/TIM2_CH1_ETR/TIM8_CHIN/ADC12_IN5/DAC2_OUT)
- new net PA6-D12-SPI1_MISO: U?.42 (PA6/SPI1_MISO/TIM8_BKIN/TIM13_CH1/DCMI_PIXCLK/TIM3_CH1/TIM1_BKIN/ADC12_IN6)
- new net PA7-D11-ETH_RMII_CRS_DV: U?.43 (PA7/SPI1_MOSI/TIM8_CH1N/TIM14_CH1/TIM3_CH2/ETH_MII_RX_DV/TIM1_CH1N/RMII_CRS_DV/ADC12_IN7)
- new net PA8-USB_HS_VBUSON: U?.100 (PA8/MCO1/USART1_CK/TIM1_CH1/I2C3_SCL/OTG_FS_SOF)
- new net PA9-OTG_FS_VBUS: U?.101 (PA9/USART1_TX/TIM1_CH2/I2C3_SMBA/DCMI_D0/OTG_FS_VBUS)
- new net PB0-USB_FS_VBUSON: U?.46 (PB0/TIM3_CH3/TIM8_CH2N/OTG_HS_ULPI_D1/ETH_MII_RXD2/TIM1_CH2N/ADC12_IN8)
- new net PB1-USB_FS_FAULT: U?.47 (PB1/TIM3_CH4/TIM8_CH3N/OTG_HS_ULPI_D2/ETH_MII_RXD3/OTG_HS_INTN/TIM1_CH3N/ADC12_IN9)
- new net PB10-SPI2_SCK-UART3_TX: U?.69 (PB10/SPI2_SCK/I2S2_CK/I2C2_SCL/USART3_TX/OTG_HS_ULPI_D3/ETH_MII_RX_ER/OTG_HS_SCL/TIM2_CH3)
- new net PB11-UART3_RX: U?.70 (PB11/I2C2_SDA/USART3_RX/OTG_HS_ULPI_D4/ETH_RMII_TX_EN/ETH_MII_TX_EN/OTG_HS_SDA/TIM2_CH4)
- new net PB12-OTG2_HS_ID: U?.73 (PB12/SPI2_NSS/I2S2_WS/I2C2_SMBA/USART3_CK/TIM1_BKIN/CAN2_RX/OTG_HS_ULPI_D5/ETH_RMII_TXD0/ETH_MII_TXD0/OTG_HS_ID)
- new net PB13-OTG_HS_VBUS: U?.74 (PB13/SPI2_SCK/I2S2_CK/USART3_CTS/TIM1_CH1N/CAN2_TX/OTG_HS_ULPI_D6/ETH_RMII_TXD1/ETH_MII_TXD1/OTG_HS_VBUS)
- new net PB14-OTG_HS_DM: U?.75 (PB14/SPI2_MISO/TIM1_CH2N/TIM12_CH1/OTG_HS_DM/USART3_RTS/TIM8_CH2N)
- new net PB15-OTG_HS_DP: U?.76 (PB15/SPI2_MOSI/I2S2_SD/TIM1_CH3N/TIM8_CH3N/TIM12_CH2/OTG_HS_DP)
- new net PB2: R3.1, U?.48 (PB2/BOOT1)
- new net PB3-TDO: U?.133 (PB3/JTDO/TRACESWO/SPI3_SCK/I2S3_CK/TIM2_CH2/SPI1_SCK)
- new net PB4-TRST: U?.134 (PB4/NJTRST/SPI3_MISO/TIM3_CH1/SPI1_MISO)
- new net PB5-D11-SPI1_MOSI: U?.135 (PB5/I2C1_SMBA/CAN2_RX/OTG_HS_ULPI_D7/ETH_PPS_OUT/TIM3_CH2/SPI1_MOSI/SPI3_MOSI/DCMI_D10/I2S3_SD)
- new net PB6-D1-USART1_TX: U?.136 (PB6/I2C1_SCL/TIM4_CH1/CAN2_TX/OTG_FS_INTN/DCMI_D5/USART1_TX)
- new net PB7-D0-USART1_RX: U?.137 (PB7/I2C1_SDA/FSMC_NL/DCMI_VSYNC/USART1_RX/TIM4_CH2)
- new net PB8-I2C1_SCL: U?.139 (PB8/TIM4_CH3/SDIO_D4/TIM10_CH1/DCMI_D6/OTG_FS_SCL/ETH_MII_TXD3/I2C1_SCL/CAN1_RX)
- new net PB9-I2C1_SDA: U?.140 (PB9/SPI2_NSS/I2S2_WS/TIM4_CH4/TIM11_CH1/OTG_FS_SDA/SDIO_D5/DCMI_D7/I2C1_SDA/CAN1_TX)
- new net PC0-A0: U?.26 (PC0/OTG_HS_ULPI_STP/ADC123_IN10)
- new net PC1-ETH_RMII_MDC: U?.27 (PC1/ETH_MDC/ADC123_IN11)
- new net PC10-SD_D2: U?.111 (PC10/SPI3_SCK/I2S3_CK/UART4_TX/SDIO_D2/DCMI_D8/USART3_TX)
- new net PC11-SD_D3: U?.112 (PC11/UART4_RX/SPI3_MISO/SDIO_D3/DCMI_D4/USART3_RX)
- new net PC12-SD_CLK: U?.113 (PC12/UART5_TX/SDIO_CK/DCMI_D9/SPI3_MOSI/I2S3_SD/USART3_CK)
- new net PC2-SPI2_MISO: U?.28 (PC2/SPI2_MISO/OTG_HS_ULPI_DIR/ETH_MII_TXD2/ADC123_IN12)
- new net PC3-SPI2_MOSI: U?.29 (PC3/SPI2_MOSI/I2S2_SD/OTG_HS_ULPI_NXT/ETH_MII_TX_CLK/ADC123_IN13)
- new net PC4-ETH_RMII_RXD0: U?.44 (PC4/ETH_RMII_RX_D0/ETH_MII_RX_D0/ADC12_IN14)
- new net PC5-ETH_RMII_RXD1: U?.45 (PC5/ETH_RMII_RX_D1/ETH_MII_RX_D1/ADC12_IN15)
- new net PC6-USART6_TX: U?.96 (PC6/SPI2_MCK/TIM8_CH1/SDIO_D6/USART6_TX/DCMI_D0/TIM3_CH1)
- new net PC7-USART6_RX: U?.97 (PC7/SPI3_MCK/TIM8_CH2/SDIO_D7/USART6_RX/DCMI_D1/TIM3_CH2)
- new net PC8-SD_D0: U?.98 (PC8/TIM8_CH3/SDIO_D0/TIM3_CH3/USART6_CK/DCMI_D2)
- new net PC9-SD_D1: U?.99 (PC9/I2S2_CKIN/I2S3_CKIN/MCO2/TIM8_CH4/SDIO_D1/I2C3_SDA/DCMI_D3/TIM3_CH4)
- new net PD0: U?.114 (PD0/FSMC_D2/CAN1_RX)
- new net PD1: U?.115 (PD1/FSMC_D3/CAN1_TX)
- new net PD10: U?.79 (PD10/FSMC_D15/USART3_CK)
- new net PD11: U?.80 (PD11/FSMC_A16/USART3_CTS)
- new net PD12: U?.81 (PD12/FSMC_A17/TIM4_CH1/USART3_RTS)
- new net PD13: U?.82 (PD13/FSMC_A18/TIM4_CH2)
- new net PD14: U?.85 (PD14/FSMC_D0/TIM4_CH3)
- new net PD15: U?.86 (PD15/FSMC_D1/TIM4_CH4)
- new net PD2-SD_CMD: U?.116 (PD2/TIM3_ETR/UART5_RX/SDIO_CMD/DCMI_D11)
- new net PD3: U?.117 (PD3/FSMC_CLK/USART2_CTS)
- new net PD4: U?.118 (PD4/FSMC_NOE/USART2_RTS)
- new net PD5: U?.119 (PD5/FSMC_NWE/USART2_TX)
- new net PD6: U?.122 (PD6/FSMC_NWAIT/USART2_RX)
- new net PD7: U?.123 (PD7/USART2_CK/FSMC_NE1/FSMC_NCE2)
- new net PD8: U?.77 (PD8/FSMC_D13/USART3_TX)
- new net PD9: U?.78 (PD9/FSMC_D14/USART3_RX)
- new net PE0: U?.141 (PE0/TIM4_ETR/FSMC_NBL0/DCMI_D2)
- new net PE1: U?.142 (PE1/FSMC_NBL1/DCMI_D3)
- new net PE2-D2: U?.1 (PE2/TRACECK/FSMC_A23/ETH_MII_TXD3)
- new net PF0: U?.10 (PF0/FSMC_A0/I2C2/SDA)
- new net PF1: U?.11 (PF1/FSMC_A1/ISC2_SCL)
- new net PF10-A5: U?.22 (PF10/FSMC_INTR/ADC3_IN8)
- new net PF11-USB_HS_FAULT: U?.49 (PF11/DCMI_12)
- new net PF12: U?.50 (PF12/FSMC_A6)
- new net PF13: U?.53 (PF13/FSMC_A7)
- new net PF14: U?.54 (PF14/FSMC_A8)
- new net PF15: U?.55 (PF15/FSMC_A9)
- new net PF2: U?.12 (PF2/FSMC_A2/I2C2_SMBA)
- new net PF3: U?.13 (PF3/FSMC_A3/ADC3_IN9)
- new net PF4: U?.14 (PF4/FSMC_A4/ADC3_IN14)
- new net PF5: U?.15 (PF5/FSMC_A5/ADC4_IN15)
- new net PF6-A1: U?.18 (PF6/TIM10_CH1/FSMC_NIORD/ADC3_IN4)
- new net PF7-A2: U?.19 (PF7/TIM11_CH1/FSMC_NREG/ADC3_IN5)
- new net PF8-A3: U?.20 (PF8/TIM13_CH1/FSMC_NIOWR/ADC3_IN6)
- new net PF9-A4: U?.21 (PF9/TIM14_CH1/FSMC_CD/ADC3_IN7)
- new net PG0: U?.56 (PG0/FSMC_A10)
- new net PG1: U?.57 (PG1/FSMC_A11)
- new net PG10-UEXT_CS: U?.125 (PG10/FSMC_NCE4_1/FSMC_NE3)
- new net PG11-ETH_RMII_TX_EN: U?.126 (PG11/FSMC_NCE4_2/ETH_MII_TX_EN)
- new net PG12-D8: U?.127 (PG12/FSMC_NE4/USART6_RTS)
- new net PG13-ETH_RMII_TXD0: U?.128 (PG13/FSMC_A24/USART6_CTS/ETH_MII_TXD0/ETH_RMII_TXD0)
- new net PG14-ETH_RMII_TXD1: U?.129 (PG14/FSMC_A25/USART6_TX/ETH_MII_TXD1/ETH_RMII_TXD1)
- new net PG15-D9: U?.132 (PG15/USART6_CTS/DCMI_D13)
- new net PG2: U?.87 (PG2/FSMC_A12)
- new net PG3: U?.88 (PG3/FSMC_A13)
- new net PG4: U?.89 (PG4/FSMC_A14)
- new net PG5: U?.90 (PG5/FSMC_A15)
- new net PG6: U?.124 (PG9/USART6_RX/FSMC_NE2/FSMC_NCE3)
- new net PG6-EPHY-RST: U?.91 (PG6/FSMC_INT2)
- new net PG7-D6: U?.92 (PG7/FSMCINT3/USART6_CK)
- new net PG8-D7: U?.93 (PG8/USART6_RTS/ETH_PPS_OUT)
- new net RST: R8.2, U?.25 (NRST)
- new net VBAT: D?.3, U?.6 (VBAT)
