File: Motion_Controller.sch (KiCad schematic (older format))
At the start: 44 parts, among them Q1 12Mhz/30ppm/20pf, Q2 32768Hz/6pF

Commit message: updated to include power and led etc
Parts:
- added C200, C35: 100nF/50V/20%/Y5V/0603, symbol Device:C_Small
- added C201: 150pF/50V/10%/0603, symbol Device:C_Small
- added C204, C205, C? (x3): 47uF/6.3V/20%/0805, symbol Device:C_Small
- added C211: 27pF/50V/5%/C0G/0603, symbol Device:C_Small
- added C60, C61: 10uF/50V/10%/1206, symbol Device:C_Small
- added Close: 3.3V_E, symbol Jumper:SolderJumper_2_Bridged
- added Close: AGND_E, symbol Jumper:SolderJumper_2_Bridged
- added D4: SMBJ26CA, symbol Device:D_Zener_Small
- added D6: 1N5822/SS34/SMA, symbol Device:D_Schottky
- added D?: LED, symbol Device:LED
- added JP?: R-T, symbol Jumper:SolderJumper_2_Open
- added JTAG: BH20R, symbol Connector_Generic:Conn_02x10_Odd_Even
- added L16: 2.2uH/1.5A/DCR<0.1R/CD32, symbol Device:L_Small
- added L19: 15uH/YS75, symbol Device:L_Small
- added PWD_JACK: PWRJ-2mm(YDJ-1134), symbol Connector:Barrel_Jack_Switch
- added PWR_LED: LED/RED/0603, symbol Device:LED
- added PWR_SEL: HN2x4(1-2:Close), symbol Connector_Generic:Conn_02x04_Odd_Even
- added R108, R85: 100k/5%/0603, symbol Device:R_Small
- added R109: NA(47k), symbol Device:R_Small
- added R26, R50, R86: 2k/1%/0603, symbol Device:R_Small
- added R30, R92: 1.1k/1%/0603, symbol Device:R_Small
- added R32: 47k/5%/0603, symbol Device:R_Small
- added R79: NA(100k), symbol Device:R_Small
- added R80: 11k/1%/0603, symbol Device:R_Small
- added R? (x9): R_Small, symbol Device:R_Small
- added R?: 4.99k/1%/0603, symbol Device:R_Small
- added SW?: WKUP, symbol Switch:SW_Push
- added U?: MP1584EN, lib_fp:SOIC-8-1EP_3.9x4.9mm_P1.27mm_EP2.29x3mm, symbol Motion_Controller:MP1584EN
- added U?: SY8009AAAC, symbol Motion_Controller:SY8009AAAC
Connections:
- net +5V: now also C35.2, C?.2, Close.2 (B), Close.2 (B), JTAG.1 (Pin_1), JTAG.2 (Pin_2), PWR_SEL.2 (Pin_2), PWR_SEL.4 (Pin_4), PWR_SEL.6 (Pin_6), PWR_SEL.8 (Pin_8), R26.2, R50.1, R?.1, R?.1, R?.1, R?.1, R?.1, SW?.1, U?.1 (EN), U?.4 (IN)
- net GNDD: now also C204.1, C205.1, C60.1, C61.1, C?.1, C?.1, C?.1, Close.1 (A), D4.2 (A), D6.2 (A), JTAG.10 (Pin_10), JTAG.12 (Pin_12), JTAG.14 (Pin_14), JTAG.16 (Pin_16), JTAG.18 (Pin_18), JTAG.20 (Pin_20), JTAG.4 (Pin_4), JTAG.6 (Pin_6), JTAG.8 (Pin_8), PWD_JACK.2, PWD_JACK.3, PWR_LED.1 (K), R108.2, R109.2, R32.1, R85.2, R86.2, R92.2, R?.1, R?.1, R?.1, R?.2, U?.2 (GND), U?.5 (GND)
- net LED: now also D?.1 (K)
- net PA0-WKUP: now also R30.1
- net PA13-TMS: now also JTAG.7 (Pin_7), R?.2
- net PA14-TCK: now also JTAG.9 (Pin_9), R?.1
- net PA15-TDI: now also JTAG.5 (Pin_5), R?.2
- net PB3-TDO: now also JTAG.13 (Pin_13), R?.2
- net PB4-TRST: now also JP?.2 (B), JTAG.3 (Pin_3), R?.2
- net RST: now also JP?.1 (A), JTAG.15 (Pin_15)
- net PE3: now reaches U?.2 (PE3/TRACED0/FSMC_A19)
- net PE4-D3: now reaches U?.3 (PE4/TRACED1/FSMC_A20/DCMI_D4)
- net PE5-D4: now reaches U?.4 (PE5/TRACED2/FSMC_A21/TIM9_CH1/DCMI_D6)
- net PE6-D5: now reaches U?.5 (PE6/TRACED3/FSMC_A22/TIM9_CH2/DCMI_D7)
- net PE7: now reaches U?.58 (PE7/FSMC_D4/TIM1_ETR)
- net PE8: now reaches U?.59 (PE8/FSMC_D5/TIM1_CH1N)
- net PE9: now reaches U?.60 (PE9/FSMC_D6/TIM1_CH1)
- net PE10: now reaches U?.63 (PE10/FSMC_D7/TIM1_CH2N)
- net PE11: now reaches U?.64 (PE11/FSMC_D8/TIM1_CH2)
- net PE12: now reaches U?.65 (PE12/FSMC_D9/TIM1_CH3N)
- net PE13: now reaches U?.66 (PE13/FSMC_D10/TIM1_CH3)
- net PE14: now reaches U?.67 (PE14/FSMC_D11/TIM1_CH4)
- net PE15: now reaches U?.68 (PE15/FSMC_D12/TIM1_BKIN)
- new net: JTAG.11 (Pin_11), R?.2, R?.2
- new net: JTAG.17 (Pin_17), R?.2
- new net: JTAG.19 (Pin_19), R?.2
- new net: C35.1, R30.2, R32.2, SW?.2
- new net: D?.2 (A), R26.1
- new net: R109.1, R79.2, U?.2 (EN)
- new net: R108.1, U?.6 (FREQ)
- new net: C200.2, L19.1, U?.1 (SW)
- new net: C201.1, U?.3 (COMP)
- new net: D6.1 (K), R80.2, R86.1, U?.4 (FB)
- new net: C200.1, U?.8 (BST)
- new net: C201.2, R85.1
- new net: L16.1, U?.3 (LX)
- new net: C211.1, R92.1, R?.2, U?.5 (FB)
- new net: C211.2, C?.2, C?.2, Close.1 (A), L16.2, R?.1
- new net: PWR_LED.2 (A), R50.2
- new net +5V_EXT: C204.2, C205.2, L19.2, PWR_SEL.1 (Pin_1), R80.1
- new net +5V_JTAG: PWR_SEL.3 (Pin_3)
- new net +5V_OTG1_PWR: PWR_SEL.7 (Pin_7)
- new net +5V_OTG2_PWR: PWR_SEL.5 (Pin_5)
- new net VSS: C60.2, C61.2, D4.1 (K), PWD_JACK.1, R79.1, U?.7 (VIN)
Other:
- note added: "BUTTON and LED"
- note added: "JTAG"
- note added: "POWER SUPPLY CIRCUIT"
- note added: "Re"
- note added: "Rf"
- note added: "STM32F407ZET6"
- note added: "Update Resistor Values"
- note added: "Vout = 0.6 x (1+Re/Rf)"
